Commit message: adding ur10 description to the simulation

File: mir_description/urdf/include/mir_100_v1.urdf.xacro (robot description, xacro)
@@ -12,4 +12,5 @@
        non-empty prefix, set prepend_prefix_to_laser_frame to 'true'. -->
   <xacro:arg name="prepend_prefix_to_laser_frame" default="false" />
+  <!--MiR-100-->
   <xacro:include filename="$(find mir_description)/urdf/include/common_properties.urdf.xacro" />
   <xacro:include filename="$(find mir_description)/urdf/include/imu.gazebo.urdf.xacro" />
@@ -17,4 +18,7 @@
   <xacro:include filename="$(find mir_description)/urdf/include/mir_100.transmission.xacro" />
   <xacro:include filename="$(find mir_description)/urdf/include/sick_s300.urdf.xacro" />
+  <!--UR1O-->
+  <xacro:include filename="$(find mir_description)/urdf/include/ur10.urdf.xacro"/>
+  <!-- <xacro:include filename="$(find mir_description)/urdf/include/cabinet.xacro"/> -->
   <xacro:property name="deg_to_rad" value="0.017453293" />
   <xacro:property name="mir_100_base_mass" value="58.0" />
@@ -224,4 +228,17 @@
     <xacro:set_all_wheel_frictions prefix="${prefix}"/>
     <xacro:p3d_base_controller prefix="${prefix}" />
+    <!--cabinet-->
+    <!-- <xacro:mmo_500_cabinet name="cabinet" parent="base_link">
+      <origin xyz="0.072 0 0.386" rpy="0 0 0" />
+    </xacro:mmo_500_cabinet> -->
+    <!--ur10-->
+    <xacro:ur10_robot parent="base_link" prefix="ur10" joint_limited="true"
+                    shoulder_pan_lower_limit="${-pi}" shoulder_pan_upper_limit="${pi}"
+                    shoulder_lift_lower_limit="${-pi}" shoulder_lift_upper_limit="${pi}"
+                    elbow_joint_lower_limit="${-pi}" elbow_joint_upper_limit="${pi}"
+                    wrist_1_lower_limit="${-pi}" wrist_1_upper_limit="${pi}"
+                    wrist_2_lower_limit="${-pi}" wrist_2_upper_limit="${pi}"
+                    wrist_3_lower_limit="${-pi}" wrist_3_upper_limit="${pi}">
+    </xacro:ur10_robot>
   </xacro:macro>
 </robot>

Commit message: adding base in description and simulation

File: mir_description/urdf/include/mir_100_v1.urdf.xacro (robot description, xacro)
@@ -20,5 +20,5 @@
   <!--UR1O-->
   <xacro:include filename="$(find mir_description)/urdf/include/ur10.urdf.xacro"/>
-  <!-- <xacro:include filename="$(find mir_description)/urdf/include/cabinet.xacro"/> -->
+  <xacro:include filename="$(find mir_description)/urdf/include/cabinet.urdf.xacro"/>
   <xacro:property name="deg_to_rad" value="0.017453293" />
   <xacro:property name="mir_100_base_mass" value="58.0" />
@@ -229,9 +229,9 @@
     <xacro:p3d_base_controller prefix="${prefix}" />
     <!--cabinet-->
-    <!-- <xacro:mmo_500_cabinet name="cabinet" parent="base_link">
-      <origin xyz="0.072 0 0.386" rpy="0 0 0" />
-    </xacro:mmo_500_cabinet> -->
+    <xacro:cabinet name="cabinet" parent="base_link">
+      <origin xyz="0.072 0 0.35" rpy="0 0 0" />
+    </xacro:cabinet>
     <!--ur10-->
-    <xacro:ur10_robot parent="base_link" prefix="ur10" joint_limited="true"
+    <xacro:ur10_robot parent="cabinet_link" prefix="ur10" joint_limited="true"
                     shoulder_pan_lower_limit="${-pi}" shoulder_pan_upper_limit="${pi}"
                     shoulder_lift_lower_limit="${-pi}" shoulder_lift_upper_limit="${pi}"

File: mir_description/urdf/include/ur10.urdf.xacro (robot description, xacro)
@@ -54,8 +54,8 @@
      wrist_2_lower_limit:=${-pi}    wrist_2_upper_limit:=${pi}
      wrist_3_lower_limit:=${-pi}    wrist_3_upper_limit:=${pi}">
-    <joint name="cabinet_u10_joint" type="fixed">
+    <joint name="cabinet_ur10_joint" type="fixed">
       <parent link="${parent}" />
       <child link = "ur10_base_link" />
-      <origin xyz="0.133 0.0 0.7" rpy="0.0 0.0 0.0" />
+      <origin xyz="0.133 0.0 0.4" rpy="0.0 0.0 0.0" />
     </joint>
     <link name="ur10_base_link" >
